File: LEC Chaser/LEC Chaser.kicad_sch (KiCad schematic)
At the start: 0 parts

Commit message: Added Latching ON/OFF circuit
Parts:
- added C1: 1u, symbol Device:C_Polarized
- added D1, D10, D2, D3, D4, D5, D6, D7, D8, D9: LED, symbol Device:LED
- added R1: 47k, symbol Device:R
- added R2: 1k, symbol Device:R
- added R3: 470R, symbol Device:R
- added U1: NE555P, Package_DIP:DIP-8_W7.62mm, symbol Timer:NE555P
- added U2: 4017, Package_DIP:DIP-16_W7.62mm, symbol 4xxx:4017
Connections:
- new net: D1.1 (K), D10.1 (K), D2.1 (K), D3.1 (K), D4.1 (K), D5.1 (K), D6.1 (K), D7.1 (K), D8.1 (K), D9.1 (K), R3.1
- new net: D10.2 (A), U2.11 (Q9)
- new net: D2.2 (A), U2.2 (Q1)
- new net: D3.2 (A), U2.4 (Q2)
- new net: C1.1, R1.2, U1.2 (TRIG), U1.6 (THRES)
- new net: R1.1, R2.2, U1.7 (DISCH)
- new net: D6.2 (A), U2.1 (Q5)
- new net: D5.2 (A), U2.10 (Q4)
- new net: D1.2 (A), U2.3 (Q0)
- new net: D7.2 (A), U2.5 (Q6)
- new net: D8.2 (A), U2.6 (Q7)
- new net: D4.2 (A), U2.7 (Q3)
- new net: D9.2 (A), U2.9 (Q8)
- new net +5V: R2.1, U1.4 (~{RST}), U1.8 (VCC), U2.16 (VDD)
- new net GND: C1.2, R3.2, U1.1 (GND), U2.13 (CKEN), U2.15 (Reset), U2.8 (VSS)
- new net NE555_OUT: U1.3 (OUT), U2.14 (CLK)
- no-connect marks 0 -> 2
